File: additions.kicad_sch (KiCad schematic)
At the start: 19 parts, among them J5 SR5-3V-200-1C, J6 SR5-3V-200-1C, J8_SW2 Conn_01x02_Pin, J8_SW3 Conn_01x02_Pin, K2 SR11-3V-200-2C, Q1 CNY74-2H, Q2 CNY74-2H

Commit message: Version 1.2
Mouser Project: https://www.mouser.com/ProjectManager/ProjectDetail.aspx?AccessID=017e74ae19
Parts:
- added J8_SW2 (x2): Conn_01x02_Pin, Connector_Phoenix_MC_HighVoltage:PhoenixContact_MCV_1,5_2-G-5.08_1x02_P5.08mm_Vertical, symbol Connector:Conn_01x02_Pin
Connections:
- net 5VDC: now also J8_SW2.1 (Pin_1)
- net COM: now also J8_SW2.2 (Pin_2)
- net at K2.5 (NO_2), R15.2: now also Q2.8 (E_1); no longer Q2.5 (E_1)
- net at J5.1 (NC): now also J8_SW2.1 (Pin_1)
- net at J5.6 (NO): no longer J8_SW2.1 (Pin_1)
- net at K2.4 (NO_1), R14.2: now also Q1.8 (E_1); no longer Q1.5 (E_1)
- net P3I renamed A3C_IN
- net A3C_IN: now also Q1.5 (E_2); no longer Q1.8 (E_2)
- net P3O renamed A3M_OUT
- net P4I renamed A4C_IN
- net A4C_IN: now also Q2.5 (E_2); no longer Q2.8 (E_2)
- net P4O renamed A4M_OUT
- new net 12COM_C: J8_SW2.2 (Pin_2)
- new net 12VDC_C: J8_SW2.1 (Pin_1)
