File: Control_board.kicad_sch (KiCad schematic)
At the start: 29 parts, among them IC1 CNY74-2H, IC2 CNY74-2H, K1 SR11-3V-200-2C, K2 SR5-12V-200-1C, U1 Teensy4.1

Commit message: V1.2 Updates
Parts:
- added D1, D2: 1N4001, Diode_THT:D_DO-41_SOD81_P10.16mm_Horizontal, symbol Diode:1N4001
- R2: value 6.19K -> 6.8K
Connections:
- net 12COM: now also D2.1 (K); no longer K2.5 (COIL_2), LED1.1 (K_GREEN_1), PS1.2 (-VIN_(GND))
- net 12VDC: now also D1.2 (A); no longer PS1.1 (+VIN_(VCC)), R2.1
- new net 12COM_C: D2.2 (A), K2.5 (COIL_2), LED1.1 (K_GREEN_1), PS1.2 (-VIN_(GND))
- new net 12VDC_C: D1.1 (K), PS1.1 (+VIN_(VCC)), R2.1
Changed lines of the file:
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@@
   (junction (at 55.88 67.31) (diameter 0) (color 0 0 0 0)
   )
+  (junction (at 152.4 26.67) (diameter 0) (color 0 0 0 0)
+  )
   (junction (at 41.91 40.64) (diameter 0) (color 0 0 0 0)
   )
@@
   (junction (at 91.44 49.53) (diameter 0) (color 0 0 0 0)
   )
+  (junction (at 148.59 22.86) (diameter 0) (color 0 0 0 0)
+  )
   (junction (at 71.12 90.17) (diameter 0) (color 0 0 0 0)
   )
@@
     (stroke (width 0) (type default))
   )
+  (wire (pts (xy 167.64 22.86) (xy 173.99 22.86))
+    (stroke (width 0) (type default))
+  )
   (wire (pts (xy 127 80.01) (xy 127 77.47))
     (stroke (width 0) (type default))
@@
     (stroke (width 0) (type default))
   )
-  (wire (pts (xy 68.58 144.78) (xy 77.47 144.78))
+  (wire (pts (xy 68.58 144.78) (xy 81.28 144.78))
     (stroke (width 0) (type default))
   )
@@
     (stroke (width 0) (type default))
   )
-  (wire (pts (xy 139.7 25.4) (xy 146.05 25.4))
-    (stroke (width 0) (type default))
-  )
   (wire (pts (xy 80.01 52.07) (xy 80.01 74.93))
     (stroke (width 0) (type default))
@@
     (stroke (width 0) (type default))
   )
+  (wire (pts (xy 152.4 26.67) (xy 148.59 26.67))
+    (stroke (width 0) (type default))
+  )
   (wire (pts (xy 55.88 35.56) (xy 66.04 35.56))
     (stroke (width 0) (type default))
@@
     (stroke (width 0) (type default))
   )
+  (wire (pts (xy 152.4 30.48) (xy 152.4 26.67))
+    (stroke (width 0) (type default))
+  )
   (wire (pts (xy 96.52 77.47) (xy 99.06 77.47))
     (stroke (width 0) (type default))
   )
+  (wire (pts (xy 148.59 17.78) (xy 148.59 22.86))
+    (stroke (width 0) (type default))
+  )
   (wire (pts (xy 82.55 77.47) (xy 55.88 77.47))
     (stroke (width 0) (type default))
   )
-  (wire (pts (xy 139.7 22.86) (xy 146.05 22.86))
-    (stroke (width 0) (type default))
-  )
   (wire (pts (xy 124.46 82.55) (xy 130.81 82.55))
     (stroke (width 0) (type default))
@@
     (stroke (width 0) (type default))
   )
+  (wire (pts (xy 139.7 22.86) (xy 148.59 22.86))
+    (stroke (width 0) (type default))
+  )
   (wire (pts (xy 209.55 93.98) (xy 214.63 93.98))
     (stroke (width 0) (type default))
@@
     (stroke (width 0) (type default))
   )
-  (wire (pts (xy 55.88 147.32) (xy 60.96 147.32))
+  (wire (pts (xy 55.88 147.32) (xy 71.12 147.32))
     (stroke (width 0) (type default))
   )
@@
     (stroke (width 0) (type default))
   )
+  (wire (pts (xy 167.64 26.67) (xy 173.99 26.67))
+    (stroke (width 0) (type default))
+  )
+  (wire (pts (xy 139.7 25.4) (xy 148.59 25.4))
+    (stroke (width 0) (type default))
+  )
   (wire (pts (xy 209.55 104.14) (xy 214.63 104.14))
     (stroke (width 0) (type default))
@@
     (stroke (width 0) (type default))
   )
+  (wire (pts (xy 148.59 22.86) (xy 160.02 22.86))
+    (stroke (width 0) (type default))
+  )
   (wire (pts (xy 55.88 137.16) (xy 60.96 137.16))
     (stroke (width 0) (type default))
@@
     (stroke (width 0) (type default))
   )
+  (wire (pts (xy 154.94 30.48) (xy 152.4 30.48))
+    (stroke (width 0) (type default))
+  )
   (wire (pts (xy 124.46 80.01) (xy 127 80.01))
     (stroke (width 0) (type default))
@@
     (stroke (width 0) (type default))
   )
+  (wire (pts (xy 160.02 26.67) (xy 152.4 26.67))
+    (stroke (width 0) (type default))
+  )
   (wire (pts (xy 153.67 153.67) (xy 160.02 153.67))
     (stroke (width 0) (type default))
@@
   )
   (wire (pts (xy 66.04 35.56) (xy 66.04 39.37))
+    (stroke (width 0) (type default))
+  )
+  (wire (pts (xy 148.59 26.67) (xy 148.59 25.4))
     (stroke (width 0) (type default))
   )
@@
     )
   )
+  (global_label "12COM_C" (shape input) (at 154.94 30.48 0) (fields_autoplaced)
+    (effects (font (size 1.27 1.27)) (justify left))
+    (property "Intersheetrefs" "${INTERSHEET_REFS}" (at 166.5543 30.48 0)
+      (effects (font (size 1.27 1.27)) (justify left) hide)
+    )
+  )
   (global_label "5VDC" (shape input) (at 92.71 22.86 180) (fields_autoplaced)
     (effects (font (size 1.27 1.27)) (justify right))
@@
     )
   )
-  (global_label "12COM" (shape input) (at 146.05 25.4 0) (fields_autoplaced)
-    (effects (font (size 1.27 1.27)) (justify left))
-    (property "Intersheetrefs" "${INTERSHEET_REFS}" (at 155.4267 25.4 0)
+  (global_label "12COM" (shape input) (at 173.99 26.67 0) (fields_autoplaced)
+    (effects (font (size 1.27 1.27)) (justify left))
+    (property "Intersheetrefs" "${INTERSHEET_REFS}" (at 183.3667 26.67 0)
       (effects (font (size 1.27 1.27)) (justify left) hide)
     )
@@
     )
   )
-  (global_label "12COM" (shape input) (at 121.92 149.86 0) (fields_autoplaced)
-    (effects (font (size 1.27 1.27)) (justify left))
-    (property "Intersheetrefs" "${INTERSHEET_REFS}" (at 131.2967 149.86 0)
+  (global_label "12VDC_C" (shape input) (at 148.59 17.78 0) (fields_autoplaced)
+    (effects (font (size 1.27 1.27)) (justify left))
+    (property "Intersheetrefs" "${INTERSHEET_REFS}" (at 159.781 17.78 0)
       (effects (font (size 1.27 1.27)) (justify left) hide)
     )
@@
     )
   )
+  (global_label "12COM_C" (shape input) (at 121.92 149.86 0) (fields_autoplaced)
+    (effects (font (size 1.27 1.27)) (justify left))
+    (property "Intersheetrefs" "${INTERSHEET_REFS}" (at 133.5343 149.86 0)
+      (effects (font (size 1.27 1.27)) (justify left) hide)
+    )
+  )
   (global_label "5VDC" (shape input) (at 160.02 148.59 0) (fields_autoplaced)
     (effects (font (size 1.27 1.27)) (justify left))
@@
     )
   )
-  (global_label "12VDC" (shape input) (at 77.47 144.78 0) (fields_autoplaced)
-    (effects (font (size 1.27 1.27)) (justify left))
-    (property "Intersheetrefs" "${INTERSHEET_REFS}" (at 86.4234 144.78 0)
-      (effects (font (size 1.27 1.27)) (justify left) hide)
-    )
-  )
-  (global_label "12VDC" (shape input) (at 146.05 22.86 0) (fields_autoplaced)
-    (effects (font (size 1.27 1.27)) (justify left))
-    (property "Intersheetrefs" "${INTERSHEET_REFS}" (at 155.0034 22.86 0)
+  (global_label "12VDC" (shape input) (at 173.99 22.86 0) (fields_autoplaced)
+    (effects (font (size 1.27 1.27)) (justify left))
+    (property "Intersheetrefs" "${INTERSHEET_REFS}" (at 182.9434 22.86 0)
       (effects (font (size 1.27 1.27)) (justify left) hide)
     )
@@
     )
   )
-  (global_label "12COM" (shape input) (at 60.96 147.32 0) (fields_autoplaced)
-    (effects (font (size 1.27 1.27)) (justify left))
-    (property "Intersheetrefs" "${INTERSHEET_REFS}" (at 70.3367 147.32 0)
+  (global_label "12COM_C" (shape input) (at 71.12 147.32 0) (fields_autoplaced)
+    (effects (font (size 1.27 1.27)) (justify left))
+    (property "Intersheetrefs" "${INTERSHEET_REFS}" (at 82.7343 147.32 0)
+      (effects (font (size 1.27 1.27)) (justify left) hide)
+    )
+  )
+  (global_label "12VDC_C" (shape input) (at 81.28 144.78 0) (fields_autoplaced)
+    (effects (font (size 1.27 1.27)) (justify left))
+    (property "Intersheetrefs" "${INTERSHEET_REFS}" (at 92.471 144.78 0)
       (effects (font (size 1.27 1.27)) (justify left) hide)
     )
@@
     (pin "47")
     (pin "48")
-    (pin "49")
     (pin "5")
-    (pin "50")
-    (pin "51")
-    (pin "52")
-    (pin "53")
-    (pin "54")
-    (pin "55")
-    (pin "56")
-    (pin "57")
-    (pin "58")
-    (pin "59")
     (pin "6")
-    (pin "60")
-    (pin "61")
-    (pin "62")
-    (pin "63")
-    (pin "64")
-    (pin "65")
-    (pin "66")
-    (pin "67")
     (pin "7")
     (pin "8")
@@
         (path "/42f06e5a-b6a6-4cd9-81d7-11930bbd2361"
           (reference "U1") (unit 1)
+        )
+      )
+    )
+  )
+  (symbol (lib_id "Diode:1N4001") (at 163.83 26.67 180) (unit 1)
+    (in_bom yes) (on_board yes) (dnp no) (fields_autoplaced)
+    (property "Reference" "D2" (at 163.83 21.59 0)
+      (effects (font (size 1.27 1.27)))
+    )
+    (property "Value" "1N4001" (at 163.83 24.13 0)
+      (effects (font (size 1.27 1.27)))
+    )
+    (property "Footprint" "Diode_THT:D_DO-41_SOD81_P10.16mm_Horizontal" (at 163.83 26.67 0)
+      (effects (font (size 1.27 1.27)) hide)
+    )
+    (property "Datasheet" "http://www.vishay.com/docs/88503/1n4001.pdf" (at 163.83 26.67 0)
+      (effects (font (size 1.27 1.27)) hide)
+    )
+    (property "Sim.Device" "D" (at 163.83 26.67 0)
+      (effects (font (size 1.27 1.27)) hide)
+    )
+    (property "Sim.Pins" "1=K 2=A" (at 163.83 26.67 0)
+      (effects (font (size 1.27 1.27)) hide)
+    )
+    (pin "1")
+    (pin "2")
+    (instances
+      (project "Control_board"
+        (path "/42f06e5a-b6a6-4cd9-81d7-11930bbd2361"
+          (reference "D2") (unit 1)
         )
       )
@@
     )
   )
+  (symbol (lib_id "Diode:1N4001") (at 163.83 22.86 0) (unit 1)
+    (in_bom yes) (on_board yes) (dnp no) (fields_autoplaced)
+    (property "Reference" "D1" (at 163.83 17.78 0)
+      (effects (font (size 1.27 1.27)))
+    )
+    (property "Value" "1N4001" (at 163.83 20.32 0)
+      (effects (font (size 1.27 1.27)))
+    )
+    (property "Footprint" "Diode_THT:D_DO-41_SOD81_P10.16mm_Horizontal" (at 163.83 22.86 0)
+      (effects (font (size 1.27 1.27)) hide)
+    )
+    (property "Datasheet" "http://www.vishay.com/docs/88503/1n4001.pdf" (at 163.83 22.86 0)
+      (effects (font (size 1.27 1.27)) hide)
+    )
+    (property "Sim.Device" "D" (at 163.83 22.86 0)
+      (effects (font (size 1.27 1.27)) hide)
+    )
+    (property "Sim.Pins" "1=K 2=A" (at 163.83 22.86 0)
+      (effects (font (size 1.27 1.27)) hide)
+    )
+    (pin "1")
+    (pin "2")
+    (instances
+      (project "Control_board"
+        (path "/42f06e5a-b6a6-4cd9-81d7-11930bbd2361"
+          (reference "D1") (unit 1)
+        )
+      )
+    )
+  )
   (symbol (lib_id "Device:R") (at 74.93 129.54 90) (unit 1)
     (in_bom yes) (on_board yes) (dnp no) (fields_autoplaced)
@@
       (effects (font (size 1.27 1.27)))
     )
-    (property "Value" "6.19K" (at 64.77 142.24 90)
-      (effects (font (size 1.27 1.27)))
-    )
+    (property "Value" "6.8K" (at 64.77 142.24 90)
+      (effects (font (size 1.27 1.27)))
+    )

Commit message: Version 1.2
Mouser Project: https://www.mouser.com/ProjectManager/ProjectDetail.aspx?AccessID=017e74ae19
Parts:
- added J1: Conn_01x02_Pin, Connector_PinHeader_2.54mm:PinHeader_1x02_P2.54mm_Vertical, symbol Connector:Conn_01x02_Pin
- added U2, U3: 01530007Z, 01530007Z, symbol SamacSys:01530007Z
Connections:
- net 12VDC_C: now also U2.2; no longer D1.1 (K)
- net 3.3V: now also U1.46 (3V3); no longer U1.15 (3V3)
- net 5VDC: now also J1.2 (Pin_2), U3.2; no longer PS1.3 (+VOUT)
- net M5V: now also J1.1 (Pin_1)
- net P3I renamed A3M_OUT
- net P3O renamed A3C_IN
- net P4I renamed A4M_OUT
- net P4O renamed A4C_IN
- new net 12VDC_A: D1.1 (K), U2.1
- new net 5VDC_A: PS1.3 (+VOUT), U3.1
Other:
- moved on the sheet: D1, D2
